File: txboardmega/txboardmega.kicad_pcb (KiCad board)
At the start: 2 copper layers, 17 parts, among them J1 Power, J10 Switch 2, J11 Switch 3, J12 Switch 4, J13 Switch 5, J14 Switch 6, J15 Encoder, J16 TX Module, J2 Display, J3 Analog 1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

Commit message: PCB update
Parts:
- added REF**: MountingHole_3.2mm_M3_DIN965, MountingHole:MountingHole_3.2mm_M3_DIN965, F.Cu at (174.0, 149.9)
- added REF**: MountingHole_3.2mm_M3_DIN965, MountingHole:MountingHole_3.2mm_M3_DIN965, F.Cu at (100.3, 149.9)
- added REF**: MountingHole_3.2mm_M3_DIN965, MountingHole:MountingHole_3.2mm_M3_DIN965, F.Cu at (174.0, 74.9)
- added REF**: MountingHole_3.2mm_M3_DIN965, MountingHole:MountingHole_3.2mm_M3_DIN965, F.Cu at (100.3, 74.9)
- moved J16 84.2 mm to (133.3, 149.9)
- moved J2 1.27 mm to (118.1, 77.5)
Connections:
- U1 pad 33: Net-(U1-Pad33) -> Net-(J9-Pad2)
- U1 pad 34: Net-(U1-Pad34) -> Net-(J10-Pad2)
- U1 pad 35: Net-(U1-Pad35) -> Net-(J11-Pad2)
- U1 pad 36: Net-(U1-Pad36) -> Net-(J12-Pad2)
- U1 pad 37: Net-(U1-Pad37) -> Net-(J13-Pad2)
- U1 pad 38: Net-(U1-Pad38) -> Net-(J14-Pad2)
Routing:
- net Net-(J1-Pad1): track 0.00 -> 216.9 mm
- net Net-(J10-Pad1): track 0.00 -> 172.6 mm
- net Net-(J15-Pad5): track 0.00 -> 82.6 mm
- net Net-(J2-Pad8): track 0.00 -> 72.3 mm
- net Net-(J15-Pad4): track 0.00 -> 66.3 mm
- net Net-(J15-Pad2): track 0.00 -> 63.8 mm
- net Net-(J9-Pad2): track 0.00 -> 40.4 mm
- net Net-(J8-Pad2): track 0.00 -> 38.8 mm
- net Net-(J3-Pad2): track 0.00 -> 33.5 mm
- net Net-(J10-Pad2): track 0.00 -> 29.7 mm
- net Net-(J7-Pad2): track 0.00 -> 29.6 mm
- net Net-(J14-Pad2): track 0.00 -> 29.3 mm
- net Net-(J4-Pad2): track 0.00 -> 27.2 mm
- net Net-(J11-Pad2): track 0.00 -> 26.7 mm
- net Net-(J6-Pad2): track 0.00 -> 26.6 mm
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Other:
- board outline added: 86.4 x 87.6 mm

Commit message: txmegaboard updates and code cleanup
Parts:
- added C1: 100nF, Capacitor_THT:C_Rect_L9.0mm_W2.5mm_P7.50mm_MKT, F.Cu at (175.8, 141.7)
- added C2: 100uF, Capacitor_THT:CP_Radial_D6.3mm_P2.50mm, F.Cu at (136.7, 150.4)
- added C3: 10uF, Capacitor_THT:CP_Radial_D5.0mm_P2.00mm, F.Cu at (145.0, 148.5)
- added R1: 10k, Resistor_THT:R_Axial_DIN0207_L6.3mm_D2.5mm_P10.16mm_Horizontal, F.Cu at (130.6, 120.4)
- added R2: 22k, Resistor_THT:R_Axial_DIN0207_L6.3mm_D2.5mm_P10.16mm_Horizontal, F.Cu at (130.6, 126.0)
- added U2: LM7809_TO220, Package_TO_SOT_THT:TO-220-3_Vertical, F.Cu at (153.9, 149.4)
- moved J15 27.9 mm to (118.1, 77.6)
- moved J2 19.2 mm to (137.3, 77.5)
- moved J16 15.5 mm to (117.9, 149.4)
Connections:
- J1 pad 1: Net-(J1-Pad1) -> Net-(C1-Pad2)
- J1 pad 2: Net-(J1-Pad2) -> Net-(C1-Pad1)
- J10 pad 1: Net-(J10-Pad1) -> Net-(C3-Pad1)
- J10 pad 3: Net-(J1-Pad1) -> Net-(C1-Pad2)
- J11 pad 1: Net-(J10-Pad1) -> Net-(C3-Pad1)
- J11 pad 3: Net-(J1-Pad1) -> Net-(C1-Pad2)
- J12 pad 1: Net-(J10-Pad1) -> Net-(C3-Pad1)
- J12 pad 3: Net-(J1-Pad1) -> Net-(C1-Pad2)
- J13 pad 1: Net-(J10-Pad1) -> Net-(C3-Pad1)
- J13 pad 3: Net-(J1-Pad1) -> Net-(C1-Pad2)
- J14 pad 1: Net-(J10-Pad1) -> Net-(C3-Pad1)
- J14 pad 3: Net-(J1-Pad1) -> Net-(C1-Pad2)
- J15 pad 1: Net-(J1-Pad1) -> Net-(C1-Pad2)
- J15 pad 3: Net-(J1-Pad1) -> Net-(C1-Pad2)
- J16 pad 2: Net-(J16-Pad2) -> Net-(C3-Pad1)
- J16 pad 3: Net-(J16-Pad3) -> Net-(C2-Pad1)
- J16 pad 4: Net-(J16-Pad4) -> Net-(C1-Pad2)
- J3 pad 1: Net-(J10-Pad1) -> Net-(C3-Pad1)
- J3 pad 3: Net-(J1-Pad1) -> Net-(C1-Pad2)
- J4 pad 1: Net-(J10-Pad1) -> Net-(C3-Pad1)
- J4 pad 3: Net-(J1-Pad1) -> Net-(C1-Pad2)
- J5 pad 1: Net-(J10-Pad1) -> Net-(C3-Pad1)
- J5 pad 3: Net-(J1-Pad1) -> Net-(C1-Pad2)
- J6 pad 1: Net-(J10-Pad1) -> Net-(C3-Pad1)
- J6 pad 3: Net-(J1-Pad1) -> Net-(C1-Pad2)
- J7 pad 1: Net-(J10-Pad1) -> Net-(C3-Pad1)
- J7 pad 3: Net-(J1-Pad1) -> Net-(C1-Pad2)
- J8 pad 1: Net-(J10-Pad1) -> Net-(C3-Pad1)
- J8 pad 3: Net-(J1-Pad1) -> Net-(C1-Pad2)
- J9 pad 1: Net-(J10-Pad1) -> Net-(C3-Pad1)
- J9 pad 3: Net-(J1-Pad1) -> Net-(C1-Pad2)
- U1 pad 1: Net-(J1-Pad2) -> Net-(C2-Pad1)
- U1 pad 16: Net-(U1-Pad16) -> Net-(J16-Pad1)
- U1 pad 2: Net-(J1-Pad2) -> Net-(C2-Pad1)
- U1 pad 20: Net-(U1-Pad20) -> Net-(J2-Pad5)
- U1 pad 21: Net-(U1-Pad21) -> Net-(J2-Pad3)
- U1 pad 3: Net-(J1-Pad1) -> Net-(C1-Pad2)
- U1 pad 4: Net-(J1-Pad1) -> Net-(C1-Pad2)
- U1 pad 5: Net-(J10-Pad1) -> Net-(C3-Pad1)
- U1 pad 6: Net-(J10-Pad1) -> Net-(C3-Pad1)
Routing:
- net Net-(C1-Pad2): track 0.00 -> 309.3 mm
- net Net-(J1-Pad1): track 216.9 -> 0.00 mm
- net Net-(C3-Pad1): track 0.00 -> 180.8 mm
- net Net-(J10-Pad1): track 172.6 -> 0.00 mm
- net Net-(J16-Pad1): track 0.00 -> 70.9 mm
- net Net-(C2-Pad1): track 0.00 -> 67.8 mm
- net Net-(C1-Pad1): track 0.00 -> 61.1 mm
- net Net-(J2-Pad5): track 0.00 -> 47.7 mm
- net Net-(J2-Pad3): track 0.00 -> 45.0 mm
- net Net-(J2-Pad6): track 0.00 -> 36.1 mm
- net Net-(J15-Pad5): track 82.6 -> 46.7 mm
- net Net-(J2-Pad7): track 0.00 -> 29.7 mm
- net Net-(J1-Pad2): track 22.6 -> 0.00 mm
- net Net-(J15-Pad2): track 63.8 -> 43.1 mm
- net Net-(J2-Pad4): track 0.00 -> 16.5 mm
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Other:
- net class Wider added: clearance 0.2, trace_width 0.5, via_dia 0.8, via_drill 0.4

Commit message: Board for Robbe Supra
Parts:
- removed C1: 100nF, Capacitor_THT:C_Rect_L9.0mm_W2.5mm_P7.50mm_MKT
- removed REF** (x4): MountingHole_3.2mm_M3_DIN965, MountingHole:MountingHole_3.2mm_M3_DIN965
- removed U2: LM7809_TO220, Package_TO_SOT_THT:TO-220-3_Vertical
- added BZ1: Buzzer, Buzzer_Beeper:Buzzer_15x7.5RM7.6, F.Cu at (166.1, 79.8)
- added J17: Trim 1, Connector_JST:JST_EH_B3B-EH-A_1x03_P2.50mm_Vertical, F.Cu at (100.6, 98.6)
- added J18: Trim 2, Connector_JST:JST_EH_B3B-EH-A_1x03_P2.50mm_Vertical, F.Cu at (100.6, 90.4)
- added J19: Trim 3, Connector_JST:JST_EH_B3B-EH-A_1x03_P2.50mm_Vertical, F.Cu at (100.6, 82.3)
- added J20: Trim 4, Connector_JST:JST_EH_B3B-EH-A_1x03_P2.50mm_Vertical, F.Cu at (100.6, 74.2)
- added J21: Bind, Connector_JST:JST_EH_B3B-EH-A_1x03_P2.50mm_Vertical, F.Cu at (134.6, 156.5)
- added K1: HF on, Relay_THT:Relay_DPDT_FRT5, F.Cu at (124.5, 142.7)
- added K2: Bind, Relay_THT:Relay_DPDT_FRT5, F.Cu at (133.1, 150.4)
- added Q1: BC107, Package_TO_SOT_THT:TO-18-3, F.Cu at (113.0, 125.0)
- added Q2: BC107, Package_TO_SOT_THT:TO-18-3, F.Cu at (113.0, 131.8)
- added R3: 10k, Resistor_THT:R_Axial_DIN0207_L6.3mm_D2.5mm_P10.16mm_Horizontal, F.Cu at (130.3, 114.8)
- added R4: 10k, Resistor_THT:R_Axial_DIN0207_L6.3mm_D2.5mm_P10.16mm_Horizontal, F.Cu at (140.5, 109.7)
- added REF1: MountingHole_3.2mm_M3_DIN965_Pad, MountingHole:MountingHole_3.2mm_M3_DIN965_Pad, F.Cu at (176.0, 158.5)
- added REF2: MountingHole_3.2mm_M3_DIN965_Pad, MountingHole:MountingHole_3.2mm_M3_DIN965_Pad, F.Cu at (99.6, 158.5)
- added REF3: MountingHole_3.2mm_M3_DIN965_Pad, MountingHole:MountingHole_3.2mm_M3_DIN965_Pad, F.Cu at (99.6, 67.3)
- added REF4: MountingHole_3.2mm_M3_DIN965_Pad, MountingHole:MountingHole_3.2mm_M3_DIN965_Pad, F.Cu at (176.0, 67.3)
- moved C2 19.5 mm to (155.4, 155.4), turned to 180 degrees
- moved J8 14.7 mm to (100.6, 109.7)
- moved J7 13.9 mm to (100.6, 117.9)
- moved J6 13.2 mm to (100.6, 126.0)
- moved J5 12.4 mm to (100.6, 134.1)
- moved J11 12.0 mm to (168.9, 122.2)
- moved J12 12.0 mm to (168.9, 113.3)
- moved J13 12.0 mm to (168.9, 104.4)
- moved J14 12.0 mm to (168.9, 95.5)
- moved J10 12.0 mm to (168.9, 131.1)
- moved J9 12.0 mm to (168.9, 140.0)
- moved J4 11.7 mm to (100.6, 142.2)
- moved J3 10.9 mm to (100.6, 150.4)
- moved C3 10.9 mm to (155.4, 145.3), turned to 180 degrees
- moved J1 10.7 mm to (166.6, 150.4)
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Connections:
- C2 pad 2: Net-(C1-Pad2) -> Net-(BZ1-Pad2)
- C3 pad 2: Net-(C1-Pad2) -> Net-(BZ1-Pad2)
- J1 pad 1: Net-(C1-Pad2) -> Net-(BZ1-Pad2)
- J1 pad 2: Net-(C1-Pad1) -> Net-(C2-Pad1)
- J10 pad 3: Net-(C1-Pad2) -> Net-(BZ1-Pad2)
- J11 pad 3: Net-(C1-Pad2) -> Net-(BZ1-Pad2)
- J12 pad 3: Net-(C1-Pad2) -> Net-(BZ1-Pad2)
- J13 pad 3: Net-(C1-Pad2) -> Net-(BZ1-Pad2)
- J14 pad 3: Net-(C1-Pad2) -> Net-(BZ1-Pad2)
- J15 pad 1: Net-(C1-Pad2) -> Net-(BZ1-Pad2)
- J15 pad 3: Net-(C1-Pad2) -> Net-(BZ1-Pad2)
- J16 pad 2: Net-(C3-Pad1) -> Net-(J16-Pad2)
- J16 pad 3: Net-(C2-Pad1) -> Net-(J16-Pad3)
- J16 pad 4: Net-(C1-Pad2) -> Net-(BZ1-Pad2)
- J3 pad 3: Net-(C1-Pad2) -> Net-(BZ1-Pad2)
- J4 pad 3: Net-(C1-Pad2) -> Net-(BZ1-Pad2)
- J5 pad 3: Net-(C1-Pad2) -> Net-(BZ1-Pad2)
- J6 pad 3: Net-(C1-Pad2) -> Net-(BZ1-Pad2)
- J7 pad 3: Net-(C1-Pad2) -> Net-(BZ1-Pad2)
- J8 pad 3: Net-(C1-Pad2) -> Net-(BZ1-Pad2)
- J9 pad 3: Net-(C1-Pad2) -> Net-(BZ1-Pad2)
- R1 pad 1: Net-(R1-Pad1) -> Net-(BZ1-Pad2)
- R1 pad 2: Net-(C1-Pad2) -> Net-(R1-Pad2)
- R2 pad 1: Net-(R1-Pad1) -> Net-(C2-Pad1)
- R2 pad 2: Net-(C1-Pad1) -> Net-(R1-Pad2)
- U1 pad 3: Net-(C1-Pad2) -> Net-(BZ1-Pad2)
- U1 pad 4: Net-(C1-Pad2) -> Net-(BZ1-Pad2)
- U1 pad 50: Net-(R1-Pad1) -> Net-(U1-Pad50)
- U1 pad 53: Net-(J15-Pad2) -> Net-(J19-Pad2)
- U1 pad 54: Net-(J15-Pad4) -> Net-(J20-Pad2)
- U1 pad 55: Net-(J15-Pad5) -> Net-(J15-Pad2)
- U1 pad 56: Net-(U1-Pad56) -> Net-(J15-Pad4)
- U1 pad 57: Net-(U1-Pad57) -> Net-(J15-Pad5)
- U1 pad 58: Net-(U1-Pad58) -> Net-(R1-Pad2)
Routing:
- net Net-(BZ1-Pad2): track 0.00 -> 348.4 mm
- net Net-(C1-Pad2): track 309.3 -> 0.00 mm
- net Net-(C3-Pad1): track 180.8 -> 243.3 mm
- net Net-(C1-Pad1): track 61.1 -> 0.00 mm
- net Net-(K2-Pad10): track 0.00 -> 61.0 mm
- net Net-(J20-Pad2): track 0.00 -> 49.7 mm
- net Net-(C2-Pad1): track 67.8 -> 109.0 mm
- net Net-(J19-Pad2): track 0.00 -> 40.1 mm
- net Net-(R1-Pad2): track 0.00 -> 37.1 mm
- net Net-(J18-Pad2): track 0.00 -> 36.9 mm
- net Net-(Q2-Pad2): track 0.00 -> 36.2 mm
- net Net-(Q1-Pad2): track 0.00 -> 34.3 mm
- net Net-(K1-Pad10): track 0.00 -> 28.9 mm
- net Net-(J17-Pad2): track 0.00 -> 28.4 mm
- net Net-(R4-Pad1): track 0.00 -> 24.0 mm
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Other:
- board size 86.4 x 87.6 mm -> 86.4 x 99.6 mm
