File: txboardmega/txboardmega.sch (KiCad schematic (older format))
At the start: 17 parts, among them J1 Power, J10 Switch 2, J11 Switch 3, J12 Switch 4, J13 Switch 5, J14 Switch 6, J15 Encoder, J16 TX Module, J2 Display, J3 Analog 1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

Commit message: PCB update
Connections:
- net at U1.33 (D22): now also J9.2 (Pin_2)
- net at U1.34 (D23): now also J10.2 (Pin_2)
- net at U1.35 (D24): now also J11.2 (Pin_2)
- net at U1.36 (D25): now also J12.2 (Pin_2)
- net at U1.37 (D26): now also J13.2 (Pin_2)
- net at U1.38 (D27): now also J14.2 (Pin_2)
Other:
- moved on the sheet: J10, J11, J12, J13, J14, J9
Changed lines of the file:
@@
 L Connector_Generic:Conn_01x03 J9
 U 1 1 6298D216
-P 9950 3900
-F 0 "J9" H 10030 3942 50  0000 L CNN
-F 1 "Switch 1" H 10030 3851 50  0000 L CNN
-F 2 "Connector_JST:JST_EH_B3B-EH-A_1x03_P2.50mm_Vertical" H 9950 3900 50  0001 C CNN
-F 3 "~" H 9950 3900 50  0001 C CNN
-	1    9950 3900
+P 2200 3200
+F 0 "J9" H 2280 3242 50  0000 L CNN
+F 1 "Switch 1" H 2280 3151 50  0000 L CNN
+F 2 "Connector_JST:JST_EH_B3B-EH-A_1x03_P2.50mm_Vertical" H 2200 3200 50  0001 C CNN
+F 3 "~" H 2200 3200 50  0001 C CNN
+	1    2200 3200
 	1    0    0    -1
 $EndComp
@@
 L Connector_Generic:Conn_01x03 J10
 U 1 1 62991DFA
-P 9950 4300
-F 0 "J10" H 10030 4342 50  0000 L CNN
-F 1 "Switch 2" H 10030 4251 50  0000 L CNN
-F 2 "Connector_JST:JST_EH_B3B-EH-A_1x03_P2.50mm_Vertical" H 9950 4300 50  0001 C CNN
-F 3 "~" H 9950 4300 50  0001 C CNN
-	1    9950 4300
+P 2200 3700
+F 0 "J10" H 2280 3742 50  0000 L CNN
+F 1 "Switch 2" H 2280 3651 50  0000 L CNN
+F 2 "Connector_JST:JST_EH_B3B-EH-A_1x03_P2.50mm_Vertical" H 2200 3700 50  0001 C CNN
+F 3 "~" H 2200 3700 50  0001 C CNN
+	1    2200 3700
 	1    0    0    -1
 $EndComp
@@
 L Connector_Generic:Conn_01x03 J11
 U 1 1 62992B4F
-P 9950 4700
-F 0 "J11" H 10030 4742 50  0000 L CNN
-F 1 "Switch 3" H 10030 4651 50  0000 L CNN
-F 2 "Connector_JST:JST_EH_B3B-EH-A_1x03_P2.50mm_Vertical" H 9950 4700 50  0001 C CNN
-F 3 "~" H 9950 4700 50  0001 C CNN
-	1    9950 4700
+P 2200 4150
+F 0 "J11" H 2280 4192 50  0000 L CNN
+F 1 "Switch 3" H 2280 4101 50  0000 L CNN
+F 2 "Connector_JST:JST_EH_B3B-EH-A_1x03_P2.50mm_Vertical" H 2200 4150 50  0001 C CNN
+F 3 "~" H 2200 4150 50  0001 C CNN
+	1    2200 4150
 	1    0    0    -1
 $EndComp
@@
 L Connector_Generic:Conn_01x03 J12
 U 1 1 62995006
-P 9950 5100
-F 0 "J12" H 10030 5142 50  0000 L CNN
-F 1 "Switch 4" H 10030 5051 50  0000 L CNN
-F 2 "Connector_JST:JST_EH_B3B-EH-A_1x03_P2.50mm_Vertical" H 9950 5100 50  0001 C CNN
-F 3 "~" H 9950 5100 50  0001 C CNN
-	1    9950 5100
+P 2200 4600
+F 0 "J12" H 2280 4642 50  0000 L CNN
+F 1 "Switch 4" H 2280 4551 50  0000 L CNN
+F 2 "Connector_JST:JST_EH_B3B-EH-A_1x03_P2.50mm_Vertical" H 2200 4600 50  0001 C CNN
+F 3 "~" H 2200 4600 50  0001 C CNN
+	1    2200 4600
 	1    0    0    -1
 $EndComp
@@
 L Connector_Generic:Conn_01x03 J13
 U 1 1 62995652
-P 9950 5500
-F 0 "J13" H 10030 5542 50  0000 L CNN
-F 1 "Switch 5" H 10030 5451 50  0000 L CNN
-F 2 "Connector_JST:JST_EH_B3B-EH-A_1x03_P2.50mm_Vertical" H 9950 5500 50  0001 C CNN
-F 3 "~" H 9950 5500 50  0001 C CNN
-	1    9950 5500
+P 2200 5050
+F 0 "J13" H 2280 5092 50  0000 L CNN
+F 1 "Switch 5" H 2280 5001 50  0000 L CNN
+F 2 "Connector_JST:JST_EH_B3B-EH-A_1x03_P2.50mm_Vertical" H 2200 5050 50  0001 C CNN
+F 3 "~" H 2200 5050 50  0001 C CNN
+	1    2200 5050
 	1    0    0    -1
 $EndComp
@@
 L Connector_Generic:Conn_01x03 J14
 U 1 1 62995DB8
-P 9950 5900
-F 0 "J14" H 10030 5942 50  0000 L CNN
-F 1 "Switch 6" H 10030 5851 50  0000 L CNN
-F 2 "Connector_JST:JST_EH_B3B-EH-A_1x03_P2.50mm_Vertical" H 9950 5900 50  0001 C CNN
-F 3 "~" H 9950 5900 50  0001 C CNN
-	1    9950 5900
-	1    0    0    -1
-$EndComp
-Text Notes 9950 3700 0    50   ~ 0
+P 2200 5500
+F 0 "J14" H 2280 5542 50  0000 L CNN
+F 1 "Switch 6" H 2280 5451 50  0000 L CNN
+F 2 "Connector_JST:JST_EH_B3B-EH-A_1x03_P2.50mm_Vertical" H 2200 5500 50  0001 C CNN
+F 3 "~" H 2200 5500 50  0001 C CNN
+	1    2200 5500
+	1    0    0    -1
+$EndComp
+Text Notes 2000 2850 0    50   ~ 0
 Switches 0-6
 $Comp
@@
 	1    0    0    -1
 $EndComp
-Wire Wire Line
-	9750 3800 9650 3800
-Wire Wire Line
-	9650 3800 9650 3200
-Connection ~ 9650 3200
-Wire Wire Line
-	9750 4200 9650 4200
-Wire Wire Line
-	9650 4200 9650 3800
-Connection ~ 9650 3800
-Wire Wire Line
-	9750 4600 9650 4600
-Wire Wire Line
-	9650 4600 9650 4200
-Connection ~ 9650 4200
-Wire Wire Line
-	9750 5000 9650 5000
-Wire Wire Line
-	9650 5000 9650 4600
-Connection ~ 9650 4600
-Wire Wire Line
-	9750 5400 9650 5400
-Wire Wire Line
-	9650 5400 9650 5000
-Connection ~ 9650 5000
-Wire Wire Line
-	9750 5800 9650 5800
-Wire Wire Line
-	9650 5800 9650 5400
-Connection ~ 9650 5400
-Wire Wire Line
-	9750 4000 9600 4000
-Wire Wire Line
-	9600 4000 9600 3400
-Connection ~ 9600 3400
-Wire Wire Line
-	9750 4400 9600 4400
-Wire Wire Line
-	9600 4400 9600 4000
-Connection ~ 9600 4000
-Wire Wire Line
-	9750 4800 9600 4800
-Wire Wire Line
-	9600 4800 9600 4400
-Connection ~ 9600 4400
-Wire Wire Line
-	9750 5200 9600 5200
-Wire Wire Line
-	9600 5200 9600 4800
-Connection ~ 9600 4800
-Wire Wire Line
-	9750 5600 9600 5600
-Wire Wire Line
-	9600 5600 9600 5200
-Connection ~ 9600 5200
-Wire Wire Line
-	9750 6000 9600 6000
-Wire Wire Line
-	9600 6000 9600 5600
-Connection ~ 9600 5600
 NoConn ~ 6100 5500
 Text Notes 1350 6950 0    50   ~ 0
@@
 Wire Wire Line
 	4500 2100 3900 2100
+Wire Wire Line
+	3900 900  1450 900
+Wire Wire Line
+	1450 900  1450 3100
+Wire Wire Line
+	1450 3100 2000 3100
+Connection ~ 3900 900
+Wire Wire Line
+	1450 3100 1450 3600
+Wire Wire Line
+	1450 3600 2000 3600
+Connection ~ 1450 3100
+Wire Wire Line
+	1450 3600 1450 4050
+Wire Wire Line
+	1450 4050 2000 4050
+Connection ~ 1450 3600
+Wire Wire Line
+	1450 4050 1450 4500
+Wire Wire Line
+	1450 4500 2000 4500
+Connection ~ 1450 4050
+Wire Wire Line
+	1450 4500 1450 4950
+Wire Wire Line
+	1450 4950 2000 4950
+Connection ~ 1450 4500
+Wire Wire Line
+	1450 4950 1450 5400
+Wire Wire Line
+	1450 5400 2000 5400
+Connection ~ 1450 4950
+Wire Wire Line
+	4000 950  1500 950
+Wire Wire Line
+	1500 950  1500 3300
+Wire Wire Line
+	1500 3300 2000 3300
+Connection ~ 4000 950
+Wire Wire Line
+	1500 3300 1500 3800
+Wire Wire Line
+	1500 3800 2000 3800
+Connection ~ 1500 3300
+Wire Wire Line
+	1500 3800 1500 4250
+Connection ~ 1500 3800
+Wire Wire Line
+	1500 4250 1500 4700
+Wire Wire Line
+	1500 4700 2000 4700
+Connection ~ 1500 4250
+Wire Wire Line
+	1500 4700 1500 5150
+Wire Wire Line
+	1500 5150 2000 5150
+Connection ~ 1500 4700
+Wire Wire Line
+	1500 5150 1500 5600
+Wire Wire Line
+	1500 5600 2000 5600
+Connection ~ 1500 5150
+Wire Wire Line
+	2000 3200 1950 3200
+Wire Wire Line
+	1950 3200 1950 3400
+Wire Wire Line
+	1950 3400 3650 3400
+Wire Wire Line
+	3650 3400 3650 4600
+Wire Wire Line
+	3650 4600 4550 4600
+Wire Wire Line
+	2000 3700 1950 3700
+Wire Wire Line
+	1950 3700 1950 3900
+Wire Wire Line
+	1950 3900 3600 3900
+Wire Wire Line
+	3600 3900 3600 4700
+Wire Wire Line
+	3600 4700 4550 4700
+Wire Wire Line
+	1500 4250 2000 4250
+Wire Wire Line
+	2000 4150 1950 4150
+Wire Wire Line
+	1950 4150 1950 4350
+Wire Wire Line
+	1950 4350 3550 4350
+Wire Wire Line
+	3550 4350 3550 4800
+Wire Wire Line
+	3550 4800 4550 4800
+Wire Wire Line
+	2000 4600 1950 4600
+Wire Wire Line
+	1950 4600 1950 4800
+Wire Wire Line
+	1950 4800 3500 4800
+Wire Wire Line
+	3500 4800 3500 4900
+Wire Wire Line
+	3500 4900 4550 4900
+Wire Wire Line
+	2000 5050 1950 5050
+Wire Wire Line
+	1950 5050 1950 5250
+Wire Wire Line
+	1950 5250 3600 5250
+Wire Wire Line
+	3600 5250 3600 5000
+Wire Wire Line
+	3600 5000 4550 5000
+Wire Wire Line
+	2000 5500 1950 5500
+Wire Wire Line
+	1950 5500 1950 5700
+Wire Wire Line
+	1950 5700 3650 5700
+Wire Wire Line
+	3650 5700 3650 5100
+Wire Wire Line
+	3650 5100 4550 5100
 $EndSCHEMATC

Commit message: txmegaboard updates and code cleanup
Parts:
- added C1: 100nF, Capacitor_THT:C_Rect_L9.0mm_W2.5mm_P7.50mm_MKT, symbol Device:C
- added C2: 100uF, Capacitor_THT:CP_Radial_D6.3mm_P2.50mm, symbol Device:CP
- added C3: 10uF, Capacitor_THT:CP_Radial_D5.0mm_P2.00mm, symbol Device:CP
- added R1: 10k, Resistor_THT:R_Axial_DIN0207_L6.3mm_D2.5mm_P10.16mm_Horizontal, symbol Device:R_Small
- added R2: 22k, Resistor_THT:R_Axial_DIN0207_L6.3mm_D2.5mm_P10.16mm_Horizontal, symbol Device:R_Small
- added U2: LM7809_TO220, Package_TO_SOT_THT:TO-220-3_Vertical, symbol Regulator_Linear:LM7808_TO220
Connections:
- net at U1.1 (Vin), U1.2 (Vin): now also J16.3 (Pin_3), C2.1, U2.3 (VO); no longer J1.2 (Pin_2)
- net at U1.16 (D5): now also J16.1 (Pin_1)
- net at U1.20 (D9): now also J2.5 (Pin_5)
- net at U1.21 (D10): now also J2.3 (Pin_3)
- net at J1.1 (Pin_1), J10.3 (Pin_3), J11.3 (Pin_3)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: now also J16.4 (Pin_4), C1.2, C2.2, C3.2, R1.2, U2.2 (GND)
- net at J10.1 (Pin_1), J11.1 (Pin_1), J12.1 (Pin_1)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: now also J16.2 (Pin_2), C3.1
- net at U1.50 (A7): now also R1.1, R2.1
- new net: C1.1, J1.2 (Pin_2), R2.2, U2.1 (VI)
- no-connect marks 1 -> 2
Other:
- note added: "+V"
- note added: "A0/DC"
- note added: "CS"
- note added: "PPM"
- note added: "Vin 10V"
- moved on the sheet: J1
Changed lines of the file:
@@
 	4550 2100 4500 2100
 Wire Wire Line
-	3900 2100 3900 6100
-Wire Wire Line
-	7450 6100 7450 5900
-Wire Wire Line
-	7450 5900 7600 5900
+	3900 2100 3900 6250
+Wire Wire Line
+	7550 5900 7600 5900
 $Comp
 L Connector_Generic:Conn_01x02 J1
 U 1 1 6292B0CC
-P 2400 1600
-F 0 "J1" H 2318 1275 50  0000 C CNN
-F 1 "Power" H 2318 1366 50  0000 C CNN
-F 2 "Connector_JST:JST_EH_B2B-EH-A_1x02_P2.50mm_Vertical" H 2400 1600 50  0001 C CNN
-F 3 "~" H 2400 1600 50  0001 C CNN
-	1    2400 1600
+P 2150 1700
+F 0 "J1" H 2068 1375 50  0000 C CNN
+F 1 "Power" H 2068 1466 50  0000 C CNN
+F 2 "Connector_JST:JST_EH_B2B-EH-A_1x02_P2.50mm_Vertical" H 2150 1700 50  0001 C CNN
+F 3 "~" H 2150 1700 50  0001 C CNN
+	1    2150 1700
 	-1   0    0    1
 $EndComp
@@
 Wire Wire Line
 	4550 1700 4500 1700
-Wire Wire Line
-	2700 1700 2700 1600
-Wire Wire Line
-	2700 1600 2600 1600
 $Comp
 L Connector_Generic:Conn_01x03 J3
@@
 Connection ~ 9600 1800
 Wire Wire Line
-	3900 6100 7450 6100
+	3900 6250 7550 6250
 Wire Wire Line
 	4550 1900 4500 1900
@@
 	3900 1900 3900 900
 Wire Wire Line
-	3900 900  9650 900
+	3900 900  7300 900
 Wire Wire Line
 	9650 900  9650 1200
 Connection ~ 9650 1200
 Wire Wire Line
-	4000 1700 4000 950
-Wire Wire Line
 	4000 950  7200 950
 Wire Wire Line
 	9600 950  9600 1400
-Connection ~ 4000 1700
-Wire Wire Line
-	4000 1700 2700 1700
 Connection ~ 9600 1400
 Text Notes 9950 1100 0    50   ~ 0
@@
 	7200 4300 7600 4300
 Wire Wire Line
-	7200 4300 7200 950
+	7200 4300 7200 3650
 Connection ~ 7200 950
 Wire Wire Line
@@
 Wire Wire Line
 	4500 1400 4500 1500
-Connection ~ 4500 1500
-Wire Wire Line
-	4500 1500 2600 1500
 Wire Wire Line
 	4550 1600 4500 1600
@@
 Connection ~ 4500 1700
 Wire Wire Line
-	4500 1700 4000 1700
-Wire Wire Line
 	4550 1800 4500 1800
 Wire Wire Line
@@
 Wire Wire Line
 	3650 5100 4550 5100
+Wire Wire Line
+	7600 3650 7200 3650
+Connection ~ 7200 3650
+Wire Wire Line
+	7200 3650 7200 2500
+Wire Wire Line
+	7600 3450 7300 3450
+Wire Wire Line
+	7300 3450 7300 900
+Connection ~ 7300 900
+Wire Wire Line
+	7300 900  9650 900
+Wire Wire Line
+	4550 2900 3950 2900
+Wire Wire Line
+	3950 2900 3950 6200
+Wire Wire Line
+	6700 6200 6700 3350
+Wire Wire Line
+	6700 3350 7600 3350
+Text Notes 7900 5450 0    50   ~ 0
+CS
+Text Notes 7900 5650 0    50   ~ 0
+A0/DC
+Wire Wire Line
+	7550 6250 7550 5900
+Wire Wire Line
+	3950 6200 6700 6200
+Wire Wire Line
+	4550 3300 4000 3300
+Wire Wire Line
+	4000 3300 4000 6150
+Wire Wire Line
+	4000 6150 7500 6150
+Wire Wire Line
+	7500 6150 7500 5600
+Wire Wire Line
+	7500 5600 7600 5600
+Wire Wire Line
+	4550 3400 4050 3400
+Wire Wire Line
+	4050 3400 4050 6100
+Wire Wire Line
+	4050 6100 7450 6100
+Wire Wire Line
+	7450 6100 7450 5400
+Wire Wire Line
+	7450 5400 7600 5400
+NoConn ~ 7600 3750
+$Comp
+L Device:R_Small R1
+U 1 1 62B96776
+P 7700 2350
+F 0 "R1" H 7759 2396 50  0000 L CNN
+F 1 "10k" H 7759 2305 50  0000 L CNN
+F 2 "Resistor_THT:R_Axial_DIN0207_L6.3mm_D2.5mm_P10.16mm_Horizontal" H 7700 2350 50  0001 C CNN
+F 3 "~" H 7700 2350 50  0001 C CNN
+	1    7700 2350
+	1    0    0    -1
+$EndComp
+$Comp
+L Device:R_Small R2
+U 1 1 62B981EC
+P 8250 2350
+F 0 "R2" H 8309 2396 50  0000 L CNN
+F 1 "22k" H 8309 2305 50  0000 L CNN
+F 2 "Resistor_THT:R_Axial_DIN0207_L6.3mm_D2.5mm_P10.16mm_Horizontal" H 8250 2350 50  0001 C CNN
+F 3 "~" H 8250 2350 50  0001 C CNN
+	1    8250 2350
+	1    0    0    -1
+$EndComp
+Text Notes 7900 3400 0    50   ~ 0
+PPM
+Text Notes 7900 3500 0    50   ~ 0
+Vcc 5V
+Text Notes 7900 3600 0    50   ~ 0
+Vin 10V
+Text Notes 7900 3700 0    50   ~ 0
+GND
+Wire Wire Line
+	6100 2100 7700 2100
+Wire Wire Line
+	7700 2100 7700 2250
+Wire Wire Line
+	8250 2250 8250 2100
+Wire Wire Line
+	8250 2100 7700 2100
+Connection ~ 7700 2100
+Wire Wire Line
+	7200 2500 7700 2500
+Wire Wire Line
+	7700 2500 7700 2450
+Connection ~ 7200 2500
+Wire Wire Line
+	7200 2500 7200 950
+Wire Wire Line
+	8500 2550 8250 2550
+Wire Wire Line
+	8250 2550 8250 2450
+Wire Wire Line
+	8500 2550 8500 1000
+Wire Wire Line
+	4500 1700 4000 1700
+Wire Wire Line
+	4000 1700 4000 950
+Connection ~ 4000 1700
+$Comp
+L Regulator_Linear:LM7808_TO220 U2
+U 1 1 62C36CF5
+P 3100 1350
+F 0 "U2" H 3100 1592 50  0000 C CNN
+F 1 "LM7809_TO220" H 3100 1501 50  0000 C CNN
+F 2 "Package_TO_SOT_THT:TO-220-3_Vertical" H 3100 1575 50  0001 C CIN
+F 3 "https://www.onsemi.cn/PowerSolutions/document/MC7800-D.PDF" H 3100 1300 50  0001 C CNN
+	1    3100 1350
+	1    0    0    -1
+$EndComp
+Wire Wire Line
+	3100 1650 3100 1700
+Connection ~ 3100 1700
+Wire Wire Line
+	2350 1600 2400 1600
+Wire Wire Line
+	2400 1600 2400 1350
+Wire Wire Line
+	2400 1350 2550 1350
+Wire Wire Line
+	3400 1350 3450 1350
+Wire Wire Line
+	4400 1350 4400 1500
+Wire Wire Line
+	4400 1500 4500 1500
+Connection ~ 4500 1500
+Wire Wire Line
+	8500 1000 2400 1000
+Wire Wire Line
+	2400 1000 2400 1350
+Connection ~ 2400 1350
+$Comp
+L Device:C C1
+U 1 1 62C6A4BD
+P 2550 1550
+F 0 "C1" H 2665 1596 50  0000 L CNN
+F 1 "100nF" H 2665 1505 50  0000 L CNN
+F 2 "Capacitor_THT:C_Rect_L9.0mm_W2.5mm_P7.50mm_MKT" H 2588 1400 50  0001 C CNN
+F 3 "~" H 2550 1550 50  0001 C CNN
+	1    2550 1550
+	1    0    0    -1
+$EndComp
+Connection ~ 2550 1700
+Wire Wire Line
+	2550 1700 2350 1700
+Wire Wire Line
+	3450 1400 3450 1350
+Wire Wire Line
+	2550 1700 3100 1700
+Connection ~ 3450 1350
+Wire Wire Line
+	3450 1350 4400 1350
+Wire Wire Line
+	2550 1400 2550 1350
+Connection ~ 2550 1350
+Wire Wire Line
+	2550 1350 2800 1350
+$Comp
+L Device:CP C3
+U 1 1 62C91123
+P 3500 1900
+F 0 "C3" V 3650 1800 50  0000 C CNN
+F 1 "10uF" V 3650 2000 50  0000 C CNN
+F 2 "Capacitor_THT:CP_Radial_D5.0mm_P2.00mm" H 3538 1750 50  0001 C CNN
+F 3 "~" H 3500 1900 50  0001 C CNN
+	1    3500 1900
+	0    1    1    0
+$EndComp
+Wire Wire Line
+	3650 1900 3900 1900
+Connection ~ 3900 1900
+Wire Wire Line
+	3100 1700 3100 1900
+Wire Wire Line
+	3100 1900 3350 1900
+Wire Wire Line
+	7600 3550 7250 3550
+Wire Wire Line
+	7250 3550 7250 1050
+Wire Wire Line
+	7250 1050 4400 1050
+Wire Wire Line
+	4400 1050 4400 1350
+Connection ~ 4400 1350
+Text Notes 1900 1750 0    50   ~ 0
+GND
+Text Notes 1950 1650 0    50   ~ 0
++V
+Wire Wire Line
+	3100 1700 3450 1700
+$Comp
+L Device:CP C2
+U 1 1 62B91980
+P 3450 1550
+F 0 "C2" H 3568 1596 50  0000 L CNN
+F 1 "100uF" H 3568 1505 50  0000 L CNN
+F 2 "Capacitor_THT:CP_Radial_D6.3mm_P2.50mm" H 3488 1400 50  0001 C CNN
+F 3 "~" H 3450 1550 50  0001 C CNN
+	1    3450 1550
+	1    0    0    -1
+$EndComp
+Connection ~ 3450 1700
+Wire Wire Line
+	3450 1700 4000 1700
 $EndSCHEMATC

Commit message: Board for Robbe Supra
Parts:
- removed C1: 100nF, Capacitor_THT:C_Rect_L9.0mm_W2.5mm_P7.50mm_MKT, symbol Device:C
- removed U2: LM7809_TO220, Package_TO_SOT_THT:TO-220-3_Vertical, symbol Regulator_Linear:LM7808_TO220
- added BZ1: Buzzer, Buzzer_Beeper:Buzzer_15x7.5RM7.6, symbol Device:Buzzer
- added J17: Trim 1, Connector_JST:JST_EH_B3B-EH-A_1x03_P2.50mm_Vertical, symbol Connector_Generic:Conn_01x03
- added J18: Trim 2, Connector_JST:JST_EH_B3B-EH-A_1x03_P2.50mm_Vertical, symbol Connector_Generic:Conn_01x03
- added J19: Trim 3, Connector_JST:JST_EH_B3B-EH-A_1x03_P2.50mm_Vertical, symbol Connector_Generic:Conn_01x03
- added J20: Trim 4, Connector_JST:JST_EH_B3B-EH-A_1x03_P2.50mm_Vertical, symbol Connector_Generic:Conn_01x03
- added J21: Bind, Connector_JST:JST_EH_B3B-EH-A_1x03_P2.50mm_Vertical, symbol Connector_Generic:Conn_01x03
- added K1: HF on, Relay_THT:Relay_DPDT_FRT5, symbol Relay:FRT5
- added K2: Bind, Relay_THT:Relay_DPDT_FRT5, symbol Relay:FRT5
- added Q1, Q2: BC107, Package_TO_SOT_THT:TO-18-3, symbol Transistor_BJT:BC107
- added R3, R4: 10k, Resistor_THT:R_Axial_DIN0207_L6.3mm_D2.5mm_P10.16mm_Horizontal, symbol Device:R_Small
Connections:
- net at C2.1, U1.1 (Vin), U1.2 (Vin): now also J1.2 (Pin_2), R2.1, K1.8; no longer J16.3 (Pin_3)
- net at U1.13 (D2): now also R3.2
- net at U1.14 (D3): now also R4.1
- net at C2.2, C3.2, J1.1 (Pin_1)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: now also R1.1, BZ1.2 (+), J17.3 (Pin_3), J18.3 (Pin_3), J19.3 (Pin_3), J20.3 (Pin_3), Q1.1 (E), Q2.1 (E); no longer R1.2
- net at U1.42 (D31): now also BZ1.1 (-)
- net at C3.1, J10.1 (Pin_1), J11.1 (Pin_1)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: now also J17.1 (Pin_1), J18.1 (Pin_1), J19.1 (Pin_1), J20.1 (Pin_1), K1.1, K1.3, K2.1; no longer J16.2 (Pin_2)
- net at U1.51 (A8): now also J17.2 (Pin_2)
- net at U1.52 (A9): now also J18.2 (Pin_2)
- net at U1.53 (A10): now also J19.2 (Pin_2); no longer J15.2 (Pin_2)
- net at U1.54 (A11): now also J20.2 (Pin_2); no longer J15.4 (Pin_4)
- net at U1.55 (A12): now also J15.2 (Pin_2); no longer J15.5 (Pin_5)
- net at U1.56 (A13): now also J15.4 (Pin_4)
- net at U1.57 (A14): now also J15.5 (Pin_5)
- net at U1.58 (A15): now also R1.2, R2.2
- new net: J16.2 (Pin_2), K1.2
- new net: J16.3 (Pin_3), K1.9
- new net: K1.10, Q2.3 (C)
- new net: K2.10, Q1.3 (C)
- new net: J21.3 (Pin_3), K2.2
- new net: J21.1 (Pin_1), K2.3
- new net: J21.2 (Pin_2), K2.4
- new net: Q2.2 (B), R3.1
- new net: Q1.2 (B), R4.2
- now unconnected: U1.50 (A7)
- no-connect marks 2 -> 7
Other:
- note added: "Analog 1-6"
- note added: "Switches 1-6"
- note added: "Trim 1-4"
- note removed: "Analog 0-5"
- note removed: "PCINT18 PK2 ADC10\nPCINT19 PK3 ADC11\nPCINT20 PK4 ADC12"
- note removed: "Switches 0-6"
- moved on the sheet: J10, J11, J12, J13, J14, J15, J16, J2, J9, R1, R2

Commit message: Added Ports and Buzzer
Parts:
- added R10, R11, R12, R13, R14, R5, R6, R7, R8, R9: 100k, Resistor_THT:R_Axial_DIN0207_L6.3mm_D2.5mm_P2.54mm_Vertical, symbol Device:R
Connections:
- net at BZ1.2 (+), C2.2, C3.2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: now also R10.1, R11.2, R12.2, R13.2, R14.2, R5.1, R6.1, R7.1, R8.1, R9.1
- net at J9.2 (Pin_2), U1.33 (D22): now also R5.2
- net at J10.2 (Pin_2), U1.34 (D23): now also R6.2
- net at J11.2 (Pin_2), U1.35 (D24): now also R7.2
- net at J12.2 (Pin_2), U1.36 (D25): now also R8.2
- net at J13.2 (Pin_2), U1.37 (D26): now also R9.2
- net at J14.2 (Pin_2), U1.38 (D27): now also R10.2
- net at J17.2 (Pin_2), U1.51 (A8): now also R11.1
- net at J18.2 (Pin_2), U1.52 (A9): now also R12.1
- net at J19.2 (Pin_2), U1.53 (A10): now also R13.1
- net at J20.2 (Pin_2), U1.54 (A11): now also R14.1
- no-connect marks 7 -> 53
